File: hardware/_saved_Belle.sch (KiCad schematic (older format))
At the start: 18 parts, among them P1 Bell CONN, P2 Battery CONN, P3 Flashing CONN, U1 74AHC1G14, U2 ESP-12, U3 AP2112

Commit message: edit layout. close #1
Parts:
- C3, C4: renamed from C?; footprint (none) -> Capacitors_SMD:C_1206_HandSoldering
Changed lines of the file:
@@
 Connection ~ 5900 2900
 $Comp
-L C_Small C?
+L C_Small C4
 U 1 1 58CE4E44
 P 8300 4300
-F 0 "C?" H 8310 4370 50  0000 L CNN
+F 0 "C4" H 8310 4370 50  0000 L CNN
 F 1 "1u" H 8310 4220 50  0000 L CNN
-F 2 "" H 8300 4300 50  0000 C CNN
+F 2 "Capacitors_SMD:C_1206_HandSoldering" H 8300 4300 50  0001 C CNN
 F 3 "" H 8300 4300 50  0000 C CNN
 	1    8300 4300
@@
 Connection ~ 8050 4300
 $Comp
-L GND #PWR?
+L GND #PWR018
 U 1 1 58CE4ED3
 P 8500 4300
-F 0 "#PWR?" H 8500 4050 50  0001 C CNN
+F 0 "#PWR018" H 8500 4050 50  0001 C CNN
 F 1 "GND" H 8500 4150 50  0000 C CNN
 F 2 "" H 8500 4300 50  0000 C CNN
@@
 	8400 4300 8500 4300
 $Comp
-L C_Small C?
+L C_Small C3
 U 1 1 58CE500B
 P 6800 4800
-F 0 "C?" H 6810 4870 50  0000 L CNN
+F 0 "C3" H 6810 4870 50  0000 L CNN
 F 1 "1u" H 6810 4720 50  0000 L CNN
-F 2 "" H 6800 4800 50  0000 C CNN
+F 2 "Capacitors_SMD:C_1206_HandSoldering" H 6800 4800 50  0001 C CNN
 F 3 "" H 6800 4800 50  0000 C CNN
 	1    6800 4800
@@
 $EndComp
 $Comp
-L GND #PWR?
+L GND #PWR019
 U 1 1 58CE504A
 P 6800 5000
-F 0 "#PWR?" H 6800 4750 50  0001 C CNN
+F 0 "#PWR019" H 6800 4750 50  0001 C CNN
 F 1 "GND" H 6800 4850 50  0000 C CNN
 F 2 "" H 6800 5000 50  0000 C CNN
