File: hardware/_autosave-Belle.kicad_pcb (KiCad board)
At the start: 2 copper layers, 44.4 x 44.5 mm, 26 parts, among them P1 Bell CONN, P2 Battery CONN, P3 FTDI Flashing CONN, P4 Boot JUMPER, U1 74AHC1G14, U2 ESP-12, U3 AP2112

Commit message: Add R9 0R resistor to layout
Parts:
- moved R3 9.69 mm to (154.9, 104.1)
Routing:
- net Net-(R3-Pad1): track 7.01 -> 25.5 mm
Other:
- board text added: "www.things.sayan.ee/belle"
- board text removed: "belle v1.0 github.com/sayanee/belle"
Changed lines of the file:
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@@
   (general
     (links 48)
-    (no_connects 3)
+    (no_connects 0)
     (area 152.324999 83.744999 196.925001 128.345001)
     (thickness 1.6)
-    (drawings 15)
-    (tracks 141)
+    (drawings 16)
+    (tracks 147)
     (zones 0)
     (modules 26)
@@
   )
   (module Resistors_SMD:R_1206_HandSoldering (layer F.Cu)
-    (at 163.195 99.06 270)
+    (at 154.94 104.14 270)
     (descr "Resistor SMD 1206, hand soldering")
     (tags "resistor 1206")
     (attr smd)
-    (fp_text reference R3 (at 4.445 0 450) (layer F.SilkS)
-      (effects (font (size 1 1) (thickness 0.15)))
-    )
-    (fp_text value 10K (at -5.08 0 450) (layer F.Fab)
+    (fp_text reference R3 (at -4.445 0 450) (layer F.SilkS)
+      (effects (font (size 1 1) (thickness 0.15)))
+    )
+    (fp_text value 10K (at 3.175 -2.54 540) (layer F.Fab)
       (effects (font (size 1 1) (thickness 0.15)))
     )
@@
     (descr "Mounting Hole 3.2mm, no annular, M3")
     (tags "mounting hole 3.2mm no annular m3")
-    (fp_text reference M3 (at -5.08 0) (layer F.SilkS)
+    (fp_text reference M3 (at 4.445 0) (layer F.SilkS)
       (effects (font (size 1 1) (thickness 0.15)))
     )
@@
     (pad 1 np_thru_hole circle (at 0 0) (size 3.2 3.2) (drill 3.2) (layers *.Cu *.Mask))
   )
+  (gr_text - (at 160.02 89.535) (layer F.SilkS)
+    (effects (font (size 1.5 1.5) (thickness 0.3)))
+  )
   (gr_text - (at 160.02 86.36) (layer F.SilkS)
     (effects (font (size 1.5 1.5) (thickness 0.3)))
@@
     (effects (font (size 1.5 1.5) (thickness 0.3)))
   )
-  (gr_text "belle v1.0 github.com/sayanee/belle" (at 174.625 107.315) (layer F.SilkS)
+  (gr_text www.things.sayan.ee/belle (at 174.625 107.315) (layer F.SilkS)
     (effects (font (size 1.5 1.5) (thickness 0.3)))
   )
@@
   (segment (start 167.64 99.725) (end 167.64 102.965) (width 0.254) (layer F.Cu) (net 7))
   (segment (start 167.64 102.965) (end 165.195 105.41) (width 0.254) (layer F.Cu) (net 7))
-  (segment (start 166.085 89.725) (end 163.195 92.615) (width 0.254) (layer F.Cu) (net 8))
+  (segment (start 167.64 89.725) (end 164.91 89.725) (width 0.254) (layer F.Cu) (net 8) (status 400000))
+  (segment (start 154.94 97.79) (end 154.94 102.14) (width 0.254) (layer F.Cu) (net 8) (status 800000))
+  (segment (start 156.21 96.52) (end 154.94 97.79) (width 0.254) (layer F.Cu) (net 8))
+  (segment (start 161.925 96.52) (end 156.21 96.52) (width 0.254) (layer F.Cu) (net 8))
+  (segment (start 163.83 94.615) (end 161.925 96.52) (width 0.254) (layer F.Cu) (net 8))
+  (segment (start 163.83 90.805) (end 163.83 94.615) (width 0.254) (layer F.Cu) (net 8))
+  (segment (start 164.91 89.725) (end 163.83 90.805) (width 0.254) (layer F.Cu) (net 8))
   (segment (start 167.64 89.725) (end 166.085 89.725) (width 0.254) (layer F.Cu) (net 8))
   (segment (start 167.64 89.725) (end 166.275 89.725) (width 0.254) (layer F.Cu) (net 8))
